Commit message: trys to fix camera orientation

File: rover_sim/models/rover_v1/model.urdf (robot description, URDF)
Before this commit: robot rover_v1, 6 links, 5 joints
Links:
- removed link back_left_wheel
- removed link back_right_wheel
- added link back_wheel, mass .2; collision cylinder length=0.02 radius=0.02; visual mesh filename=package://ugv_sim/meshes/wheel.stl scale=0.15 0.15 0.15
- link camera_link: mass 0.0 -> 0.05; geometry collision box size=.01 0.01 0.01; visual box size=.01 0.01 0.01
- link left_wheel: geometry collision cylinder length=0.02 radius=0.02; visual mesh filename=package://ugv_sim/meshes/wheel.stl scale=0.15 0.15 0.15
- link right_wheel: geometry collision cylinder length=0.02 radius=0.02; visual mesh filename=package://ugv_sim/meshes/wheel.stl scale=0.15 0.15 0.15
Joints:
- removed joint back_left_joint
- removed joint back_right_joint
- added joint back_wheel_joint: type continuous, parent base_link, child back_wheel, origin xyz=0.0 .04 -0.05 rpy=0 0 -1.5708, axis 0 1 0
- joint camera_joint: axis 0 1 0 -> (none); limit lower=0 upper=0 effort=0 velocity=0 -> (none); origin xyz=0.0  .04  0.0 rpy=0 0 1.5708 -> xyz=0.0  -.065  0.0 rpy=0 0 -1.5708
- joint left_joint: origin xyz=-0.13 .04 -0.05 rpy=0 0 -1.5708 -> xyz=-0.12 -.04 -0.05 rpy=0 0 -1.5708
- joint right_joint: origin xyz=0.13 .04 -0.05 rpy=0 0 -1.5708 -> xyz=0.12 -.04 -0.05 rpy=0 0 -1.5708
