Commit message: adds a (not working) IMU sensor to the rover sim

File: rover_sim/models/rover_v2/model.urdf (robot description, URDF)
Before this commit: robot rover_v2, 6 links, 5 joints
Links:
- added link imu_link, mass 0.05; collision box size=0.1 0.1 0.1; visual box size=0.1 0.1 0.1
Joints:
- added joint imu_joint: type fixed, parent base_link, child imu_link, origin xyz=0.0  0.0  0.0 rpy=0 0 -1.5708

Commit message: fixes "missing" wheel.stl

File: rover_sim/models/rover_v2/model.urdf (robot description, URDF)
Before this commit: robot rover_v2, 7 links, 6 joints
Links:
- link back_wheel: geometry collision cylinder length=0.02 radius=0.02; visual mesh filename=package://rover_sim/models/rover_v2/meshes/wheel.stl scale=0.15 0.15 0.15
- link left_wheel: geometry collision cylinder length=0.02 radius=0.02; visual mesh filename=package://rover_sim/models/rover_v2/meshes/wheel.stl scale=0.15 0.15 0.15
- link right_wheel: geometry collision cylinder length=0.02 radius=0.02; visual mesh filename=package://rover_sim/models/rover_v2/meshes/wheel.stl scale=0.15 0.15 0.15
