Commit message: updats to revision 3 of rover model

File: rover_sim/models/rover_v3/model.urdf (robot description, URDF)
Before this commit: robot rover_v3, 6 links, 5 joints
Links:
- link base_link: geometry collision box size=.120 .20 .11; visual box size=.120 .20 .11
Joints:
- joint back_wheel_joint: origin xyz=0.0 .06 -0.05 rpy=0 0 -1.5708 -> xyz=-.06 0.0 -0.05 rpy=0 0 0
- joint camera_joint: origin xyz=0.0  -.065  0.0 rpy=0 0 -1.5708 -> xyz=0.0  -.065  0.0 rpy=0 0 0
- joint left_joint: origin xyz=-0.1325 -.015 -0.030 rpy=0 0 -1.5708 -> xyz=.015 -0.1325 -0.030 rpy=0 0 0
- joint right_joint: origin xyz=0.1325 -.015 -0.030 rpy=0 0 -1.5708 -> xyz=.015 0.1325 -0.030 rpy=0 0 0

Commit message: refinements to model

File: rover_sim/models/rover_v3/model.urdf (robot description, URDF)
Before this commit: robot rover_v3, 6 links, 5 joints
Joints:
- joint left_joint: origin xyz=-0.1325 -.015 -0.030 rpy=0 0 -1.5708 -> xyz=0.1325 -.015 -0.030 rpy=0 0 -1.5708
- joint right_joint: origin xyz=0.1325 -.015 -0.030 rpy=0 0 -1.5708 -> xyz=-0.1325 -.015 -0.030 rpy=0 0 -1.5708

Commit message: sets rover in final configuration

File: rover_sim/models/rover_v3/model.urdf (robot description, URDF)
Before this commit: robot rover_v3, 6 links, 5 joints
Links:
- link back_wheel: mass .2 -> .05
- link base_link: geometry collision box size=.2 .12 .11; visual box size=.2 .12 .11
Joints:
- joint back_wheel_joint: origin xyz=-.06 0.0 -0.05 rpy=0 0 0 -> xyz=-.1 0.0 -0.055 rpy=0 0 0
- joint camera_joint: origin xyz=0.0  -.065  0.0 rpy=0 0 0 -> xyz=0.105 0.0 0.0 rpy=0 0 0
- joint left_joint: origin xyz=0.1325 -.015 -0.030 rpy=0 0 -1.5708 -> xyz=0.05 0.1 -0.030 rpy=0 0 0
- joint right_joint: origin xyz=-0.1325 -.015 -0.030 rpy=0 0 -1.5708 -> xyz=0.05 -0.1 -0.030 rpy=0 0 0

Commit message: adds imu_link

File: rover_sim/models/rover_v3/model.urdf (robot description, URDF)
Before this commit: robot rover_v3, 6 links, 5 joints
Links:
- added link imu_link, mass 0.05; collision box size=.01 0.01 0.01; visual box size=.01 0.01 0.01
Joints:
- added joint imu_joint: type fixed, parent base_link, child imu_link, origin xyz=0.105 0.0 0.0 rpy=0 0 0

Commit message: makes the sim model drivable again

File: rover_sim/models/rover_v3/model.urdf (robot description, URDF)
Before this commit: robot rover_v3, 7 links, 6 joints
Links:
- removed link back_wheel
- added link caster_link, mass .2; collision sphere radius=.03; visual sphere radius=.03
- link base_link: mass 1.242 -> 2.5
Joints:
- removed joint back_wheel_joint
- added joint caster_joint: type continuous, parent base_link, child caster_link, origin xyz=-0.05  0   -0.055 rpy=0 0 0
